Commit message: Update roid1.urdf

File: urdf/roid1.urdf (robot description, URDF)
Before this commit: robot roid1, 24 links, 23 joints
Links:
- link c_chest: geometry visual mesh filename=package://roid1_urdf/urdf/c_chest_a.stl; visual mesh filename=package://roid1_urdf/urdf/c_chest_b.stl
- link c_head: geometry visual mesh filename=package://roid1_urdf/urdf/c_head_a.stl; visual mesh filename=package://roid1_urdf/urdf/c_head_b.stl
- link c_waist: geometry visual mesh filename=package://roid1_urdf/urdf/c_waist.stl
- link foot_r: geometry visual mesh filename=package://roid1_urdf/urdf/r_foot.stl
- link l_ankle: geometry visual mesh filename=package://roid1_urdf/urdf/l_ankle.stl
- link l_elbow: geometry visual mesh filename=package://roid1_urdf/urdf/l_elbow.stl
- link l_foot: geometry visual mesh filename=package://roid1_urdf/urdf/l_foot.stl
- link l_hipjointlower: geometry visual mesh filename=package://roid1_urdf/urdf/l_hipjointlower.stl
- link l_hipjointupper: geometry visual mesh filename=package://roid1_urdf/urdf/l_hipjointupper.stl; visual mesh filename=package://roid1_urdf/urdf/l_hipjointupperpoint.stl
- link l_lowerarm: geometry visual mesh filename=package://roid1_urdf/urdf/l_lowerarm.stl
- link l_lowerreg: geometry visual mesh filename=package://roid1_urdf/urdf/l_lowerreg_a.stl; visual mesh filename=package://roid1_urdf/urdf/l_lowerreg_b.stl
- link l_shoulder: geometry visual mesh filename=package://roid1_urdf/urdf/l_shoulder.stl; visual mesh filename=package://roid1_urdf/urdf/shoulderpoint.stl
- link l_uppararm: geometry visual mesh filename=package://roid1_urdf/urdf/l_upperarm.stl
- link l_upperreg: geometry visual mesh filename=package://roid1_urdf/urdf/l_upperreg_a.stl; visual mesh filename=package://roid1_urdf/urdf/l_upperreg_b.stl
- link r_ankle: geometry visual mesh filename=package://roid1_urdf/urdf/r_ankle.stl
- link r_elbow: geometry visual mesh filename=package://roid1_urdf/urdf/r_elbow.stl
- link r_hipjointlower: geometry visual mesh filename=package://roid1_urdf/urdf/r_hipjointlower.stl
- link r_hipjointupper: geometry visual mesh filename=package://roid1_urdf/urdf/r_hipjointupper.stl; visual mesh filename=package://roid1_urdf/urdf/r_hipjointupperpoint.stl
- link r_lowerarm: geometry visual mesh filename=package://roid1_urdf/urdf/r_lowerarm.stl
- link r_lowerreg: geometry visual mesh filename=package://roid1_urdf/urdf/r_lowerreg_a.stl; visual mesh filename=package://roid1_urdf/urdf/r_lowerreg_b.stl
- link r_shoulder: geometry visual mesh filename=package://roid1_urdf/urdf/r_shoulder.stl; visual mesh filename=package://roid1_urdf/urdf/shoulderpoint.stl
- link r_uppararm: geometry visual mesh filename=package://roid1_urdf/urdf/r_upperarm.stl
- link r_upperreg: geometry visual mesh filename=package://roid1_urdf/urdf/r_upperreg_a.stl; visual mesh filename=package://roid1_urdf/urdf/r_upperreg_b.stl

Commit message: Renamed some links

File: urdf/roid1.urdf (robot description, URDF)
Before this commit: robot roid1, 24 links, 23 joints
Links:
- removed link foot_r
- removed link l_uppararm
- removed link r_uppararm
- added link l_upperarm; visual mesh filename=package://roid1_urdf/urdf/l_upperarm.stl
- added link r_foot; visual mesh filename=package://roid1_urdf/urdf/r_foot.stl
- added link r_upperarm; visual mesh filename=package://roid1_urdf/urdf/r_upperarm.stl
Joints:
- joint l_elbow_yaw: parent l_uppararm -> l_upperarm
- joint l_shoulder_roll: child l_uppararm -> l_upperarm
- joint r_ankle_roll: child foot_r -> r_foot
- joint r_elbow_yaw: parent r_uppararm -> r_upperarm
- joint r_shoulder_roll: child r_uppararm -> r_upperarm

Commit message: Update roid1.urdf
File name fixed

File: urdf/roid1.urdf (robot description, URDF)
Before this commit: robot roid1, 24 links, 23 joints
Links:
- removed link l_lowerreg
- removed link l_upperreg
- removed link r_lowerreg
- removed link r_upperreg
- added link l_lowerleg; visual mesh filename=package://roid1_urdf/urdf/l_lowerleg_a.stl; visual mesh filename=package://roid1_urdf/urdf/l_lowerleg_b.stl
- added link l_upperleg; visual mesh filename=package://roid1_urdf/urdf/l_upperleg_a.stl; visual mesh filename=package://roid1_urdf/urdf/l_upperleg_b.stl
- added link r_lowerleg; visual mesh filename=package://roid1_urdf/urdf/r_lowerleg_a.stl; visual mesh filename=package://roid1_urdf/urdf/r_lowerleg_b.stl
- added link r_upperleg; visual mesh filename=package://roid1_urdf/urdf/r_upperleg_a.stl; visual mesh filename=package://roid1_urdf/urdf/r_upperleg_b.stl
Joints:
- joint l_ankle_pitch: parent l_lowerreg -> l_lowerleg
- joint l_hipjoint_pitch: child l_upperreg -> l_upperleg
- joint l_knee_pitch: child l_lowerreg -> l_lowerleg; parent l_upperreg -> l_upperleg
- joint r_ankle_pitch: parent r_lowerreg -> r_lowerleg
- joint r_hipjoint_pitch: child r_upperreg -> r_upperleg
- joint r_knee_pitch: child r_lowerreg -> r_lowerleg; parent r_upperreg -> r_upperleg
